File: i960SxProcessorMegaShieldFormFactor.sch (KiCad schematic (older format))
At the start: 31 parts, among them P1 Power, P2 Data Lines Lower, P3 Data Lines Upper, P4 Address Lines, P5 PWM, P6 Serializable Pins, P7 1284p Direct Connection, U1 74HC245, U2 74HC245, U3 80960Sx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

Commit message: link up pre-existing external hardware
Fix errors and make sure we are using AHC parts
Parts:
- added R3, R4: 10k, Resistor_SMD:R_0805_2012Metric_Pad1.20x1.40mm_HandSolder, symbol Device:R
Connections:
- net +5V: now also R3.1, R4.1
- net ~INT0: now also R4.2
- net ~INT3: now also R3.2
- net ~READY: no longer U3.79 (READY_)
- net MCU_FAIL: now reaches P5.3 (Pin_3)
- new net ~READY960: U3.79 (READY_)
- no-connect marks 7 -> 6
Other:
- moved on the sheet: D1, R2
Changed lines of the file:
@@
 $Descr A3 16535 11693
 encoding utf-8
-Sheet 1 1
+Sheet 1 2
 Title "i960Sx Mega Shield Without direct connection to a mega"
-Date "2021-05-08"
-Rev "1"
+Date "2021-10-20"
+Rev "2"
 Comp "Joshua Scoggins"
 Comment1 "No Serialization Hardware"
-Comment2 "No Synchronization Hardware"
+Comment2 "Synchronization Hardware included"
 Comment3 ""
 Comment4 ""
@@
 L Device:R R2
 U 1 1 6DFEA54A
-P 15350 7850
-F 0 "R2" V 15143 7850 50  0000 C CNN
-F 1 "560" V 15234 7850 50  0000 C CNN
-F 2 "Resistor_SMD:R_0805_2012Metric_Pad1.20x1.40mm_HandSolder" V 15280 7850 50  0001 C CNN
-F 3 "~" H 15350 7850 50  0001 C CNN
-	1    15350 7850
-	1    0    0    -1
-$EndComp
-Wire Wire Line
-	15350 7700 15350 7050
+P 1550 7150
+F 0 "R2" V 1343 7150 50  0000 C CNN
+F 1 "560" V 1434 7150 50  0000 C CNN
+F 2 "Resistor_SMD:R_0805_2012Metric_Pad1.20x1.40mm_HandSolder" V 1480 7150 50  0001 C CNN
+F 3 "~" H 1550 7150 50  0001 C CNN
+	1    1550 7150
+	1    0    0    -1
+$EndComp
+Wire Wire Line
+	1550 7000 1550 6350
 $Comp
 L Device:LED D1
 U 1 1 6E0899FD
-P 15350 6900
-F 0 "D1" H 15343 6645 50  0000 C CNN
-F 1 "POWER LED" H 15343 6736 50  0000 C CNN
-F 2 "LED_SMD:LED_0805_2012Metric" H 15350 6900 50  0001 C CNN
-F 3 "~" H 15350 6900 50  0001 C CNN
-	1    15350 6900
+P 1550 6200
+F 0 "D1" H 1543 5945 50  0000 C CNN
+F 1 "POWER LED" H 1543 6036 50  0000 C CNN
+F 2 "LED_SMD:LED_0805_2012Metric" H 1550 6200 50  0001 C CNN
+F 3 "~" H 1550 6200 50  0001 C CNN
+	1    1550 6200
 	0    1    1    0
 $EndComp
 Wire Wire Line
-	15350 6750 15350 6450
-Wire Wire Line
-	15350 8000 15350 8300
-Wire Wire Line
-	15350 8300 14650 8300
+	1550 6050 1550 5750
+Wire Wire Line
+	1550 7300 1550 7600
+Wire Wire Line
+	1550 7600 850  7600
 $Comp
 L power:+3.3V #PWR012
 U 1 1 6E1C9DB5
-P 14650 8300
-F 0 "#PWR012" H 14650 8150 50  0001 C CNN
-F 1 "+3.3V" H 14665 8473 50  0000 C CNN
-F 2 "" H 14650 8300 50  0001 C CNN
-F 3 "" H 14650 8300 50  0001 C CNN
-	1    14650 8300
+P 850 7600
+F 0 "#PWR012" H 850 7450 50  0001 C CNN
+F 1 "+3.3V" H 865 7773 50  0000 C CNN
+F 2 "" H 850 7600 50  0001 C CNN
+F 3 "" H 850 7600 50  0001 C CNN
+	1    850  7600
 	0    -1   -1   0
 $EndComp
@@
 L power:GND #PWR013
 U 1 1 6E129E38
-P 15350 6450
-F 0 "#PWR013" H 15350 6200 50  0001 C CNN
-F 1 "GND" H 15355 6277 50  0000 C CNN
-F 2 "" H 15350 6450 50  0001 C CNN
-F 3 "" H 15350 6450 50  0001 C CNN
-	1    15350 6450
+P 1550 5750
+F 0 "#PWR013" H 1550 5500 50  0001 C CNN
+F 1 "GND" H 1555 5577 50  0000 C CNN
+F 2 "" H 1550 5750 50  0001 C CNN
+F 3 "" H 1550 5750 50  0001 C CNN
+	1    1550 5750
 	0    -1   -1   0
 $EndComp
@@
 D15
 Text Label 6750 4000 2    50   ~ 0
-~READY
+~READY960
 Text Label 6750 3900 2    50   ~ 0
 ALE
@@
 $EndComp
 NoConn ~ 13750 1200
-NoConn ~ 15250 1350
 NoConn ~ 15250 1250
 NoConn ~ 15250 1150
@@
 	15100 2150 15100 1450
 Wire Wire Line
-	15000 1350 15250 1350
-Wire Wire Line
 	15250 1250 15000 1250
 Wire Wire Line
@@
 Wire Wire Line
 	9500 4900 9500 6400
+Wire Wire Line
+	15000 1350 15700 1350
+Text Label 15700 1350 2    50   ~ 0
+MCU_FAIL
+$Sheet
+S 13500 7500 900  600
+U 62305776
+F0 "Sheet62305775" 50
+F1 "ExternalHardware.sch" 50
+F2 "~READY960" O R 14400 7600 50
+F3 "MCU_FAIL" O R 14400 7700 50
+F4 "~READY" I L 13500 7600 50
+F5 "CLKO" I L 13500 7700 50
+F6 "~BLAST~\\~FAIL~" I L 13500 7800 50
+F7 "~BE1" I L 13500 7900 50
+F8 "~BE0" I L 13500 8000 50
+$EndSheet
+Text Label 12750 7600 0    50   ~ 0
+~READY
+Wire Wire Line
+	12750 7600 13500 7600
+Wire Wire Line
+	13500 7700 12750 7700
+Wire Wire Line
+	13500 7800 12750 7800
+Wire Wire Line
+	13500 7900 12750 7900
+Wire Wire Line
+	13500 8000 12750 8000
+Wire Wire Line
+	15150 7600 14400 7600
+Wire Wire Line
+	15150 7700 14400 7700
+Text Label 15150 7600 2    50   ~ 0
+~READY960
+Text Label 15150 7700 2    50   ~ 0
+MCU_FAIL
+Text Label 12750 7700 0    50   ~ 0
+CLKO
+Text Label 12750 7800 0    50   ~ 0
+~BLAST~\~FAIL~
+Text Label 12750 8000 0    50   ~ 0
+~BE0
+Text Label 12750 7900 0    50   ~ 0
+~BE1
+$Comp
+L Device:R R4
+U 1 1 6243CF68
+P 6750 9700
+F 0 "R4" H 6820 9746 50  0000 L CNN
+F 1 "10k" H 6820 9655 50  0000 L CNN
+F 2 "Resistor_SMD:R_0805_2012Metric_Pad1.20x1.40mm_HandSolder" V 6680 9700 50  0001 C CNN
+F 3 "~" H 6750 9700 50  0001 C CNN
+	1    6750 9700
+	1    0    0    -1
+$EndComp
+Wire Wire Line
+	6750 9850 6750 10200
+Wire Wire Line
+	6750 10200 7450 10200
+Wire Wire Line
+	6750 9550 6750 9300
+Text Label 7450 10200 2    50   ~ 0
+~INT0
+$Comp
+L power:+5V #PWR?
+U 1 1 624853C2
+P 6750 9300
+AR Path="/629FB5E8/624853C2" Ref="#PWR?"  Part="1"
+AR Path="/624853C2" Ref="#PWR017"  Part="1"
+F 0 "#PWR017" H 6750 9150 50  0001 C CNN
+F 1 "+5V" H 6765 9473 50  0000 C CNN
+F 2 "" H 6750 9300 50  0001 C CNN
+F 3 "" H 6750 9300 50  0001 C CNN
+	1    6750 9300
+	1    0    0    -1
+$EndComp
+$Comp
+L Device:R R3
+U 1 1 62485C2F
+P 5450 10350
+F 0 "R3" H 5520 10396 50  0000 L CNN
+F 1 "10k" H 5520 10305 50  0000 L CNN
+F 2 "Resistor_SMD:R_0805_2012Metric_Pad1.20x1.40mm_HandSolder" V 5380 10350 50  0001 C CNN
+F 3 "~" H 5450 10350 50  0001 C CNN
+	1    5450 10350
+	1    0    0    -1
+$EndComp
+Wire Wire Line
+	5450 10500 5450 10850
+Wire Wire Line
+	5450 10850 6150 10850
+Wire Wire Line
+	5450 10200 5450 9950
+$Comp
+L power:+5V #PWR?
+U 1 1 62485C38
+P 5450 9950
+AR Path="/629FB5E8/62485C38" Ref="#PWR?"  Part="1"
+AR Path="/62485C38" Ref="#PWR016"  Part="1"
+F 0 "#PWR016" H 5450 9800 50  0001 C CNN
+F 1 "+5V" H 5465 10123 50  0000 C CNN
+F 2 "" H 5450 9950 50  0001 C CNN
+F 3 "" H 5450 9950 50  0001 C CNN
+	1    5450 9950
+	1    0    0    -1
+$EndComp
+Text Label 6150 10850 2    50   ~ 0
+~INT3
 $EndSCHEMATC

Commit message: Move the transceivers and registers to make room for the aux hardware
Connections:
- net A10: now also P4.15 (Pin_15); no longer P4.23 (Pin_23)
- net A11: now also P4.16 (Pin_16); no longer P4.24 (Pin_24)
- net A12: now also P4.13 (Pin_13); no longer P4.21 (Pin_21)
- net A13: now also P4.14 (Pin_14); no longer P4.22 (Pin_22)
- net A14: now also P4.11 (Pin_11); no longer P4.19 (Pin_19)
- net A15: now also P4.12 (Pin_12); no longer P4.20 (Pin_20)
- net A8: now also P4.17 (Pin_17); no longer P4.25 (Pin_25)
- net A9: now also P4.18 (Pin_18); no longer P4.26 (Pin_26)
- net AD1: now also U2.8 (A6); no longer U2.3 (A1)
- net AD10: now also U1.7 (A5); no longer U1.4 (A2)
- net AD11: now also U1.6 (A4); no longer U1.5 (A3)
- net AD12: now also U1.5 (A3); no longer U1.6 (A4)
- net AD13: now also U1.4 (A2); no longer U1.7 (A5)
- net AD14: now also U1.3 (A1); no longer U1.8 (A6)
- net AD15: now also U1.2 (A0); no longer U1.9 (A7)
- net AD2: now also U2.7 (A5); no longer U2.4 (A2)
- net AD3: now also U2.6 (A4); no longer U2.5 (A3)
- net AD4: now also U2.5 (A3); no longer U2.6 (A4)
- net AD5: now also U2.4 (A2); no longer U2.7 (A5)
- net AD6: now also U2.3 (A1); no longer U2.8 (A6)
- net AD7: now also U2.2 (A0); no longer U2.9 (A7)
- net AD8: now also U1.9 (A7); no longer U1.2 (A0)
- net AD9: now also U1.8 (A6); no longer U1.3 (A1)
- net D0: now also U2.9 (A7); no longer U2.2 (A0)
- net D0_OUT: now also P4.25 (Pin_25), U2.11 (B7); no longer P4.17 (Pin_17), U2.18 (B0)
- net D1: now also P4.26 (Pin_26), U2.12 (B6); no longer P4.18 (Pin_18), U2.17 (B1)
- net D10: now also U1.13 (B5); no longer U1.16 (B2)
- net D11: now also U1.14 (B4); no longer U1.15 (B3)
- net D12: now also U1.15 (B3); no longer U1.14 (B4)
- net D13: now also U1.16 (B2); no longer U1.13 (B5)
- net D14: now also U1.17 (B1); no longer U1.12 (B6)
- net D15: now also U1.18 (B0); no longer U1.11 (B7)
- net D2: now also P4.23 (Pin_23), U2.13 (B5); no longer P4.15 (Pin_15), U2.16 (B2)
- net D3: now also P4.24 (Pin_24), U2.14 (B4); no longer P4.16 (Pin_16), U2.15 (B3)
- net D4: now also P4.21 (Pin_21), U2.15 (B3); no longer P4.13 (Pin_13), U2.14 (B4)
- net D5: now also P4.22 (Pin_22), U2.16 (B2); no longer P4.14 (Pin_14), U2.13 (B5)
- net D6: now also P4.19 (Pin_19), U2.17 (B1); no longer P4.11 (Pin_11), U2.12 (B6)
- net D7: now also P4.20 (Pin_20), U2.18 (B0); no longer P4.12 (Pin_12), U2.11 (B7)
- net D8: now also U1.11 (B7); no longer U1.18 (B0)
- net D9: now also U1.12 (B6); no longer U1.17 (B1)

Commit message: Mostly complete rewiring
Parts:
- added R?: 10k, Resistor_SMD:R_0805_2012Metric_Pad1.20x1.40mm_HandSolder, symbol Device:R
Connections:
- net +5V: now also R?.1
- net ~RESET960: now also R?.2
Changed lines of the file:
@@
 Wire Wire Line
 	3950 8550 2600 8550
+$Comp
+L Device:R R?
+U 1 1 627A8D7D
+P 8750 10300
+F 0 "R?" H 8820 10346 50  0000 L CNN
+F 1 "10k" H 8820 10255 50  0000 L CNN
+F 2 "Resistor_SMD:R_0805_2012Metric_Pad1.20x1.40mm_HandSolder" V 8680 10300 50  0001 C CNN
+F 3 "~" H 8750 10300 50  0001 C CNN
+	1    8750 10300
+	1    0    0    -1
+$EndComp
+Wire Wire Line
+	8750 10450 8750 10800
+Wire Wire Line
+	8750 10800 9450 10800
+Wire Wire Line
+	8750 10150 8750 9900
+$Comp
+L power:+5V #PWR?
+U 1 1 627A8D86
+P 8750 9900
+AR Path="/629FB5E8/627A8D86" Ref="#PWR?"  Part="1"
+AR Path="/627A8D86" Ref="#PWR?"  Part="1"
+F 0 "#PWR?" H 8750 9750 50  0001 C CNN
+F 1 "+5V" H 8765 10073 50  0000 C CNN
+F 2 "" H 8750 9900 50  0001 C CNN
+F 3 "" H 8750 9900 50  0001 C CNN
+	1    8750 9900
+	1    0    0    -1
+$EndComp
+Text Label 9450 10800 2    50   ~ 0
+~RESET960
 $EndSCHEMATC

Commit message: Save the added pullup resistor
Parts:
- gave numbers to parts that had none: 1
Changed lines of the file:
@@
 	3950 8550 2600 8550
 $Comp
-L Device:R R?
+L Device:R R7
 U 1 1 627A8D7D
 P 8750 10300
-F 0 "R?" H 8820 10346 50  0000 L CNN
+F 0 "R7" H 8820 10346 50  0000 L CNN
 F 1 "10k" H 8820 10255 50  0000 L CNN
 F 2 "Resistor_SMD:R_0805_2012Metric_Pad1.20x1.40mm_HandSolder" V 8680 10300 50  0001 C CNN
@@
 P 8750 9900
 AR Path="/629FB5E8/627A8D86" Ref="#PWR?"  Part="1"
-AR Path="/627A8D86" Ref="#PWR?"  Part="1"
-F 0 "#PWR?" H 8750 9750 50  0001 C CNN
+AR Path="/627A8D86" Ref="#PWR0101"  Part="1"
+F 0 "#PWR0101" H 8750 9750 50  0001 C CNN
 F 1 "+5V" H 8765 10073 50  0000 C CNN
 F 2 "" H 8750 9900 50  0001 C CNN

Commit message: Put the data and address lines back into the previous design
Maximizes compatibility?
Connections:
- net A10: now also P4.23 (Pin_23); no longer P4.15 (Pin_15)
- net A11: now also P4.24 (Pin_24); no longer P4.16 (Pin_16)
- net A12: now also P4.21 (Pin_21); no longer P4.13 (Pin_13)
- net A13: now also P4.22 (Pin_22); no longer P4.14 (Pin_14)
- net A14: now also P4.19 (Pin_19); no longer P4.11 (Pin_11)
- net A15: now also P4.20 (Pin_20); no longer P4.12 (Pin_12)
- net A8: now also P4.25 (Pin_25); no longer P4.17 (Pin_17)
- net A9: now also P4.26 (Pin_26); no longer P4.18 (Pin_18)
- net D0_OUT: now also P4.17 (Pin_17); no longer P4.25 (Pin_25)
- net D1: now also P4.18 (Pin_18); no longer P4.26 (Pin_26)
- net D2: now also P4.15 (Pin_15); no longer P4.23 (Pin_23)
- net D3: now also P4.16 (Pin_16); no longer P4.24 (Pin_24)
- net D4: now also P4.13 (Pin_13); no longer P4.21 (Pin_21)
- net D5: now also P4.14 (Pin_14); no longer P4.22 (Pin_22)
- net D6: now also P4.11 (Pin_11); no longer P4.19 (Pin_19)
- net D7: now also P4.12 (Pin_12); no longer P4.20 (Pin_20)
Changed lines of the file:
@@
 ~BE1
 NoConn ~ 13450 1550
-Text Label 14250 5650 1    50   ~ 0
-A15
-Text Label 14350 5650 1    50   ~ 0
-A13
-Text Label 14450 5650 1    50   ~ 0
-A11
-Text Label 14550 5650 1    50   ~ 0
-A9
-Text Label 15050 5650 1    50   ~ 0
-A7
-Text Label 15150 5650 1    50   ~ 0
-A5
-Text Label 15250 5650 1    50   ~ 0
-A3
-Text Label 15350 5650 1    50   ~ 0
-A1
-Text Label 13850 5650 1    50   ~ 0
-D15
-Text Label 13950 5650 1    50   ~ 0
-D13
-Text Label 14050 5650 1    50   ~ 0
-D11
-Text Label 14150 5650 1    50   ~ 0
-D9
-Text Label 14650 5650 1    50   ~ 0
-D7
-Text Label 14750 5650 1    50   ~ 0
-D5
-Text Label 14850 5650 1    50   ~ 0
-D3
-Text Label 14950 5650 1    50   ~ 0
-D1
-Text Label 14250 4650 1    50   ~ 0
+Text Label 14650 4650 1    50   ~ 0
 A14
-Text Label 14350 4650 1    50   ~ 0
+Text Label 14750 4650 1    50   ~ 0
 A12
-Text Label 14450 4650 1    50   ~ 0
+Text Label 14850 4650 1    50   ~ 0
 A10
-Text Label 14550 4650 1    50   ~ 0
+Text Label 14950 4650 1    50   ~ 0
 A8
 Text Label 15050 4650 1    50   ~ 0
@@
 Text Label 15350 4650 1    50   ~ 0
 A0
-Text Label 13850 4650 1    50   ~ 0
-D14
-Text Label 13950 4650 1    50   ~ 0
-D12
-Text Label 14050 4650 1    50   ~ 0
-D10
-Text Label 14150 4650 1    50   ~ 0
-D8
-Text Label 14650 4650 1    50   ~ 0
-D6
-Text Label 14750 4650 1    50   ~ 0
-D4
-Text Label 14850 4650 1    50   ~ 0
-D2
-Text Label 14950 4650 1    50   ~ 0
-D0_OUT
 $Comp
 L Connector_Generic:Conn_02x18_Odd_Even P4
@@
 $EndComp
 Wire Wire Line
-	14250 4850 14250 4650
-Wire Wire Line
-	14350 4850 14350 4650
-Wire Wire Line
-	14450 4850 14450 4650
-Wire Wire Line
-	14550 4850 14550 4650
-Wire Wire Line
 	15050 4850 15050 4650
 Wire Wire Line
@@
 	15350 4850 15350 4650
 Wire Wire Line
-	13850 4850 13850 4650
-Wire Wire Line
-	13950 4850 13950 4650
-Wire Wire Line
-	14050 4850 14050 4650
-Wire Wire Line
-	14150 4850 14150 4650
-Wire Wire Line
 	14650 4850 14650 4650
 Wire Wire Line
@@
 Wire Wire Line
 	14950 4850 14950 4650
-Wire Wire Line
-	14250 5350 14250 5650
-Wire Wire Line
-	14350 5350 14350 5650
-Wire Wire Line
-	14450 5350 14450 5650
-Wire Wire Line
-	14550 5350 14550 5650
-Wire Wire Line
-	15050 5350 15050 5650
-Wire Wire Line
-	15150 5350 15150 5650
-Wire Wire Line
-	15250 5350 15250 5650
-Wire Wire Line
-	15350 5350 15350 5650
-Wire Wire Line
-	13850 5350 13850 5650
-Wire Wire Line
-	13950 5350 13950 5650
-Wire Wire Line
-	14050 5350 14050 5650
-Wire Wire Line
-	14150 5350 14150 5650
-Wire Wire Line
-	14650 5350 14650 5650
-Wire Wire Line
-	14750 5350 14750 5650
-Wire Wire Line
-	14950 5350 14950 5650
-Wire Wire Line
-	14850 5350 14850 5650
 Text Label 13750 2450 0    50   ~ 0
 A31
@@
 Text Label 9450 10800 2    50   ~ 0
 ~RESET960
+Wire Wire Line
+	14150 4850 14150 4650
+Wire Wire Line
+	14050 4850 14050 4650
+Wire Wire Line
+	13950 4850 13950 4650
+Wire Wire Line
+	13850 4850 13850 4650
+Wire Wire Line
+	14550 4850 14550 4650
+Wire Wire Line
+	14450 4850 14450 4650
+Wire Wire Line
+	14350 4850 14350 4650
+Wire Wire Line
+	14250 4850 14250 4650
+Text Label 14550 4650 1    50   ~ 0
+D0_OUT
+Text Label 14450 4650 1    50   ~ 0
+D2
+Text Label 14350 4650 1    50   ~ 0
+D4
+Text Label 14250 4650 1    50   ~ 0
+D6
+Text Label 14150 4650 1    50   ~ 0
+D8
+Text Label 14050 4650 1    50   ~ 0
+D10
+Text Label 13950 4650 1    50   ~ 0
+D12
+Text Label 13850 4650 1    50   ~ 0
+D14
+Wire Wire Line
+	15350 5350 15350 5650
+Wire Wire Line
+	15250 5350 15250 5650
+Wire Wire Line
+	15150 5350 15150 5650
+Wire Wire Line
+	15050 5350 15050 5650
+Wire Wire Line
+	14950 5350 14950 5650
+Wire Wire Line
+	14850 5350 14850 5650
+Wire Wire Line
+	14750 5350 14750 5650
+Wire Wire Line
+	14650 5350 14650 5650
+Text Label 15350 5650 1    50   ~ 0
+A1
+Text Label 15250 5650 1    50   ~ 0
+A3
+Text Label 15150 5650 1    50   ~ 0
+A5
+Text Label 15050 5650 1    50   ~ 0
+A7
+Text Label 14950 5650 1    50   ~ 0
+A9
+Text Label 14850 5650 1    50   ~ 0
+A11
+Text Label 14750 5650 1    50   ~ 0
+A13
+Text Label 14650 5650 1    50   ~ 0
+A15
+Wire Wire Line
+	14450 5350 14450 5650
+Wire Wire Line
+	14550 5350 14550 5650
+Wire Wire Line
+	14350 5350 14350 5650
+Wire Wire Line
+	14250 5350 14250 5650
+Wire Wire Line
+	14150 5350 14150 5650
+Wire Wire Line
+	14050 5350 14050 5650
+Wire Wire Line
+	13950 5350 13950 5650
+Wire Wire Line
+	13850 5350 13850 5650
+Text Label 14550 5650 1    50   ~ 0
+D1
+Text Label 14450 5650 1    50   ~ 0
+D3
+Text Label 14350 5650 1    50   ~ 0
+D5
+Text Label 14250 5650 1    50   ~ 0
+D7
+Text Label 14150 5650 1    50   ~ 0
+D9
+Text Label 14050 5650 1    50   ~ 0
+D11
+Text Label 13950 5650 1    50   ~ 0
+D13
+Text Label 13850 5650 1    50   ~ 0
+D15
 $EndSCHEMATC

Commit message: expose clock signal div 2
Connections:
- net CLK_DIV2: now reaches P5.1 (Pin_1)
- no-connect marks 6 -> 5
Changed lines of the file:
@@
 NoConn ~ 13750 1200
 NoConn ~ 15250 1250
-NoConn ~ 15250 1150
 Wire Wire Line
 	15000 1550 15700 1550
@@
 Wire Wire Line
 	15250 1250 15000 1250
-Wire Wire Line
-	15000 1150 15250 1150
 Connection ~ 14100 1950
 Wire Wire Line
@@
 F7 "~BE1" I L 13500 7900 50
 F8 "~BE0" I L 13500 8000 50
+F9 "CLKDIV2" O R 14400 7800 50
 $EndSheet
 Text Label 12750 7600 0    50   ~ 0
@@
 Text Label 13850 5650 1    50   ~ 0
 D15
+Wire Wire Line
+	15000 1150 15700 1150
+Text Label 15700 1150 2    50   ~ 0
+CLK_DIV2
+Wire Wire Line
+	14400 7800 15150 7800
+Text Label 15150 7800 2    50   ~ 0
+CLK_DIV2
 $EndSCHEMATC

Commit message: Connect MCU_RDY to ~READY pin
In the old designs, the ~READY pin was never used outside of the stack
and the ~MCU_RDY pin was used in its place. I want to now make it so
that using ~READY will always be synchronized. But the older rev1 cards
directly connect ready to the i960Sx
Connections:
- net ~READY: now also P5.2 (Pin_2)
- no-connect marks 5 -> 4
Changed lines of the file:
@@
 $EndComp
 NoConn ~ 13750 1200
-NoConn ~ 15250 1250
 Wire Wire Line
 	15000 1550 15700 1550
@@
 Wire Wire Line
 	15100 2150 15100 1450
-Wire Wire Line
-	15250 1250 15000 1250
 Connection ~ 14100 1950
 Wire Wire Line
@@
 Text Label 15150 7800 2    50   ~ 0
 CLK_DIV2
+Wire Wire Line
+	15000 1250 15700 1250
+Text Label 15700 1250 2    50   ~ 0
+~READY
 $EndSCHEMATC
