File: i960SxProcessorMegaShieldFormFactor.kicad_sch (KiCad schematic)
At the start: 36 parts, among them P1 Power, P2 Data Lines Lower, P3 Data Lines Upper, P4 Address Lines, P5 PWM, P6 Serializable Pins, P7 1284p Direct Connection, U1 74LVC16T245, U2 74AHC16373, U3 80960Sx

Commit message: Remove the external hardware sheet
We want to keep this board as simple as possible

Having the extra signal setups is not a smart move it seems
Connections:
- net ~{READY960} is gone; now on net ~{READY}: U3.79 (READY_)
- net ~{READY}: now also P5.6 (Pin_6); no longer P5.2 (Pin_2)
- net MCU_FAIL: no longer names the net of P5.3 (Pin_3)
- no-connect marks 6 -> 7
Other:
- removed sheet Sheet62305775
Changed lines of the file:
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@@
   (junction (at 396.24 123.19) (diameter 0) (color 0 0 0 0)
   )
+  (no_connect (at 398.78 34.29))
   (no_connect (at 349.25 30.48))
   (no_connect (at 398.78 39.37))
-  (no_connect (at 398.78 41.91))
   (no_connect (at 341.63 39.37))
   (no_connect (at 360.68 34.29))
+  (no_connect (at 398.78 31.75))
   (no_connect (at 398.78 29.21))
   (wire (pts (xy 381 46.99) (xy 398.78 46.99))
@@
     (stroke (width 0) (type default) (color 0 0 0 0))
   )
-  (wire (pts (xy 342.9 203.2) (xy 323.85 203.2))
-    (stroke (width 0) (type default) (color 0 0 0 0))
-  )
   (wire (pts (xy 93.98 85.09) (xy 63.5 85.09))
     (stroke (width 0) (type default) (color 0 0 0 0))
@@
     (stroke (width 0) (type default) (color 0 0 0 0))
   )
-  (wire (pts (xy 384.81 195.58) (xy 365.76 195.58))
-    (stroke (width 0) (type default) (color 0 0 0 0))
-  )
   (wire (pts (xy 257.81 203.2) (xy 289.56 203.2))
     (stroke (width 0) (type default) (color 0 0 0 0))
@@
     (stroke (width 0) (type default) (color 0 0 0 0))
   )
-  (wire (pts (xy 342.9 198.12) (xy 323.85 198.12))
-    (stroke (width 0) (type default) (color 0 0 0 0))
-  )
   (wire (pts (xy 359.41 123.19) (xy 359.41 118.11))
     (stroke (width 0) (type default) (color 0 0 0 0))
@@
     (stroke (width 0) (type default) (color 0 0 0 0))
   )
-  (wire (pts (xy 342.9 200.66) (xy 323.85 200.66))
-    (stroke (width 0) (type default) (color 0 0 0 0))
-  )
   (wire (pts (xy 93.98 44.45) (xy 63.5 44.45))
     (stroke (width 0) (type default) (color 0 0 0 0))
@@
     (stroke (width 0) (type default) (color 0 0 0 0))
   )
-  (wire (pts (xy 323.85 193.04) (xy 342.9 193.04))
-    (stroke (width 0) (type default) (color 0 0 0 0))
-  )
   (wire (pts (xy 255.27 177.8) (xy 289.56 177.8))
     (stroke (width 0) (type default) (color 0 0 0 0))
@@
     (stroke (width 0) (type default) (color 0 0 0 0))
   )
-  (wire (pts (xy 342.9 195.58) (xy 323.85 195.58))
-    (stroke (width 0) (type default) (color 0 0 0 0))
-  )
   (wire (pts (xy 396.24 123.19) (xy 392.43 123.19))
     (stroke (width 0) (type default) (color 0 0 0 0))
@@
     (stroke (width 0) (type default) (color 0 0 0 0))
   )
-  (wire (pts (xy 384.81 193.04) (xy 365.76 193.04))
-    (stroke (width 0) (type default) (color 0 0 0 0))
-  )
   (wire (pts (xy 57.15 252.73) (xy 57.15 240.03))
     (stroke (width 0) (type default) (color 0 0 0 0))
@@
     (effects (font (size 1.27 1.27)) (justify right bottom))
   )
-  (label "~{READY960}" (at 384.81 193.04 180)
-    (effects (font (size 1.27 1.27)) (justify right bottom))
-  )
   (label "A13" (at 374.65 143.51 90)
     (effects (font (size 1.27 1.27)) (justify left bottom))
@@
     (effects (font (size 1.27 1.27)) (justify left bottom))
   )
-  (label "CLKO" (at 323.85 195.58 0)
-    (effects (font (size 1.27 1.27)) (justify left bottom))
-  )
   (label "AD12" (at 63.5 92.71 0)
     (effects (font (size 1.27 1.27)) (justify left bottom))
@@
     (effects (font (size 1.27 1.27)) (justify left bottom))
   )
-  (label "~{READY}" (at 323.85 193.04 0)
-    (effects (font (size 1.27 1.27)) (justify left bottom))
-  )
   (label "D11" (at 356.87 143.51 90)
     (effects (font (size 1.27 1.27)) (justify left bottom))
@@
     (effects (font (size 1.27 1.27)) (justify right bottom))
   )
-  (label "~{BE0}" (at 323.85 203.2 0)
-    (effects (font (size 1.27 1.27)) (justify left bottom))
-  )
   (label "AD10" (at 63.5 97.79 0)
     (effects (font (size 1.27 1.27)) (justify left bottom))
@@
     (effects (font (size 1.27 1.27)) (justify right bottom))
   )
-  (label "~{BE1}" (at 323.85 200.66 0)
-    (effects (font (size 1.27 1.27)) (justify left bottom))
-  )
   (label "D13" (at 190.5 162.56 0)
     (effects (font (size 1.27 1.27)) (justify left bottom))
@@
     (effects (font (size 1.27 1.27)) (justify right bottom))
   )
-  (label "MCU_FAIL" (at 384.81 195.58 180)
-    (effects (font (size 1.27 1.27)) (justify right bottom))
-  )
   (label "A1" (at 297.18 91.44 180)
     (effects (font (size 1.27 1.27)) (justify right bottom))
@@
     (effects (font (size 1.27 1.27)) (justify left bottom))
   )
-  (label "~{BLAST}\\~{FAIL}" (at 323.85 198.12 0)
-    (effects (font (size 1.27 1.27)) (justify left bottom))
-  )
   (label "A19" (at 349.25 96.52 0)
     (effects (font (size 1.27 1.27)) (justify left bottom))
   )
-  (label "MCU_FAIL" (at 398.78 34.29 180)
-    (effects (font (size 1.27 1.27)) (justify right bottom))
-  )
   (label "D7" (at 361.95 143.51 90)
     (effects (font (size 1.27 1.27)) (justify left bottom))
@@
     (effects (font (size 1.27 1.27)) (justify right bottom))
   )
-  (label "~{READY}" (at 398.78 31.75 180)
+  (label "~{READY}" (at 398.78 41.91 180)
     (effects (font (size 1.27 1.27)) (justify right bottom))
   )
@@
     (effects (font (size 1.27 1.27)) (justify left bottom))
   )
-  (label "~{READY960}" (at 171.45 101.6 180)
+  (label "~{READY}" (at 171.45 101.6 180)
     (effects (font (size 1.27 1.27)) (justify right bottom))
   )
@@
     (pin "1")
   )
-  (sheet (at 342.9 190.5) (size 22.86 15.24) (fields_autoplaced)
-    (stroke (width 0) (type solid) (color 0 0 0 0))
-    (fill (color 0 0 0 0.0000))
-    (property "Sheet name" "Sheet62305775" (id 0) (at 342.9 189.7884 0)
-      (effects (font (size 1.27 1.27)) (justify left bottom))
-    )
-    (property "Sheet file" "ExternalHardware.kicad_sch" (id 1) (at 342.9 206.3246 0)
-      (effects (font (size 1.27 1.27)) (justify left top))
-    )
-    (pin "~{READY960}" output (at 365.76 193.04 0)
-      (effects (font (size 1.27 1.27)) (justify right))
-    )
-    (pin "MCU_FAIL" output (at 365.76 195.58 0)
-      (effects (font (size 1.27 1.27)) (justify right))
-    )
-    (pin "~{READY}" input (at 342.9 193.04 180)
-      (effects (font (size 1.27 1.27)) (justify left))
-    )
-    (pin "CLKO" input (at 342.9 195.58 180)
-      (effects (font (size 1.27 1.27)) (justify left))
-    )
-    (pin "~{BLAST}\\~{FAIL}" input (at 342.9 198.12 180)
-      (effects (font (size 1.27 1.27)) (justify left))
-    )
-    (pin "~{BE1}" input (at 342.9 200.66 180)
-      (effects (font (size 1.27 1.27)) (justify left))
-    )
-    (pin "~{BE0}" input (at 342.9 203.2 180)
-      (effects (font (size 1.27 1.27)) (justify left))
-    )
-  )
   (sheet_instances
     (path "/" (page "1"))
-    (path "/00000000-0000-0000-0000-000062305776" (page "2"))
   )
   (symbol_instances
@@
       (reference "#PWR017") (unit 1) (value "+5V") (footprint "")
     )
-    (path "/00000000-0000-0000-0000-000062305776/99f7fbf9-d3be-41ae-bb93-06b2ddb925f2"
-      (reference "#PWR018") (unit 1) (value "+5V") (footprint "")
-    )
-    (path "/00000000-0000-0000-0000-000062305776/b4a36e75-b869-4c47-b59c-ca31346a3bd7"
-      (reference "#PWR019") (unit 1) (value "GND") (footprint "")
-    )
     (path "/77dea360-5400-44ac-8c9a-e88cec47a5a2"
       (reference "#PWR020") (unit 1) (value "VCC") (footprint "")
@@
       (reference "#PWR026") (unit 1) (value "GND") (footprint "")
     )
-    (path "/00000000-0000-0000-0000-000062305776/0e2482b9-a689-45a3-a536-674e09a602a2"
-      (reference "#PWR028") (unit 1) (value "+5V") (footprint "")
-    )
-    (path "/00000000-0000-0000-0000-000062305776/ea681034-3b40-4892-8a79-d88436b1d240"
-      (reference "#PWR029") (unit 1) (value "GND") (footprint "")
-    )
     (path "/fceec026-2774-410a-a23d-28afe3dbe1f1"
       (reference "#PWR030") (unit 1) (value "GND") (footprint "")
@@
       (reference "#PWR044") (unit 1) (value "VCC") (footprint "")
     )
-    (path "/00000000-0000-0000-0000-000062305776/54d67715-4a9a-43b7-87fd-557773a7b7f7"
-      (reference "#PWR045") (unit 1) (value "+5V") (footprint "")
-    )
     (path "/00000000-0000-0000-0000-0000627a8d86"
       (reference "#PWR0101") (unit 1) (value "+5V") (footprint "")
@@
       (reference "C16") (unit 1) (value "0.1uF") (footprint "Capacitor_SMD:C_0805_2012Metric_Pad1.18x1.45mm_HandSolder")
     )
-    (path "/00000000-0000-0000-0000-000062305776/8ac9015a-d982-42ad-ab7f-11cd1a812831"
-      (reference "C17") (unit 1) (value "0.1uF") (footprint "Capacitor_SMD:C_0805_2012Metric_Pad1.18x1.45mm_HandSolder")
-    )
     (path "/d01a0665-1937-43dc-82a6-6500e620f7b7"
       (reference "C18") (unit 1) (value "0.1uF") (footprint "Capacitor_SMD:C_0805_2012Metric_Pad1.18x1.45mm_HandSolder")
     )
-    (path "/00000000-0000-0000-0000-000062305776/37cf12d2-9997-4855-9d67-d21913190832"
-      (reference "C19") (unit 1) (value "0.1uF") (footprint "Capacitor_SMD:C_0805_2012Metric_Pad1.18x1.45mm_HandSolder")
-    )
     (path "/c4879764-615c-43d9-8e12-d4c5af018cdc"
       (reference "C20") (unit 1) (value "0.1uF") (footprint "Capacitor_SMD:C_0805_2012Metric_Pad1.18x1.45mm_HandSolder")
@@
       (reference "R4") (unit 1) (value "10k") (footprint "Resistor_SMD:R_0805_2012Metric_Pad1.20x1.40mm_HandSolder")
     )
-    (path "/00000000-0000-0000-0000-000062305776/ba417558-e07a-4aa8-8f8c-15d6dc468305"
-      (reference "R6") (unit 1) (value "10k") (footprint "Resistor_SMD:R_0805_2012Metric_Pad1.20x1.40mm_HandSolder")
-    )
     (path "/00000000-0000-0000-0000-0000627a8d7d"
       (reference "R7") (unit 1) (value "10k") (footprint "Resistor_SMD:R_0805_2012Metric_Pad1.20x1.40mm_HandSolder")
@@
       (reference "U3") (unit 1) (value "80960Sx") (footprint "Package_LCC:PLCC-84_THT-Socket")
     )
-    (path "/00000000-0000-0000-0000-000062305776/67f3f848-2b47-48d4-8ef6-b211a1c5ad8a"
-      (reference "U7") (unit 1) (value "74AHC74") (footprint "Package_SO:SOIC-14_3.9x8.7mm_P1.27mm")
-    )
-    (path "/00000000-0000-0000-0000-000062305776/3d5d3e16-fe05-4ff3-a365-9890d25e1af0"
-      (reference "U7") (unit 3) (value "74AHC74") (footprint "Package_SO:SOIC-14_3.9x8.7mm_P1.27mm")
-    )
-    (path "/00000000-0000-0000-0000-000062305776/312ed157-03e4-4f79-8162-ee244f6128f1"
-      (reference "U8") (unit 1) (value "GAL16V8") (footprint "Package_LCC:PLCC-20_THT-Socket")
-    )
   )
